Commit message: Fix the knee bending backwards in the humanoid models
Knee's range (-60..+5 deg) made it swing the shank forward: a bird's
knee, on both legs, so the mirror fix in #402 couldn't catch it. The knee
axis is flipped in whole_body_humanoid.urdf and in the Pioneer v2 robot
(pioneer_humanoid_v2.urdf, pioneer_v2.xml), so negative Knee now bends the
knee with the foot going back. The ranges are unchanged.

The Isaac Lab default stance (Hip_F 0.12, Knee -0.22) put the feet about
18 cm in front of the hips with the old sign. With the fix they sit under
the hips; Ankle_P goes to -0.10 and Ankle_R to +0.04 to keep the soles
level. Policies trained on the old knee are not valid on this one.

check_leg_directions.py checks that each leg joint moves the way a
person's does (Hip_F the knee forward, Hip_A out, Knee the ankle back,
Ankle_P the toes down). The old URDF fails both knees; the fixed models
pass 8 of 8.

Co-Authored-By: Wilson Cheng <150957380+wilsonchenghy@users.noreply.github.com>

File: assets/pioneer_v2_humanoid/pioneer_humanoid_v2.urdf (robot description, URDF)
Before this commit: robot pioneer_humanoid_v2, 70 links, 69 joints
Joints:
- joint Knee_L: axis 1.000000 0.000000 0.000000 -> -1.000000 0.000000 0.000000
- joint Knee_R: axis 1.000000 0.000000 0.000000 -> -1.000000 0.000000 0.000000
