Commit message: Whole-body humanoid: limit the elbows to their real bend (-90..0 deg)
l_elbow / r_elbow were -90..+90 deg, but only the negative side bends the arm the way an elbow can
(the hand comes forward); positive angles folded the forearm backwards past straight. Upper limit set
to 0 in the URDF and the MJCF regenerated with to_mjcf.py (only the 4 elbow lines change).
check_motion.py: every joint moves cleanly.

Co-Authored-By: Claude Opus 5.5 <noreply@anthropic.com>

File: assets/pioneer_whole_body_humanoid/pioneer_whole_body_humanoid.urdf (robot description, URDF)
Before this commit: robot pioneer_whole_body_humanoid, 70 links, 69 joints
Joints:
- joint l_elbow: limit lower=-1.5708 upper=1.5708 effort=22 velocity=6 -> lower=-1.5708 upper=0 effort=22 velocity=6
- joint r_elbow: limit lower=-1.5708 upper=1.5708 effort=22 velocity=6 -> lower=-1.5708 upper=0 effort=22 velocity=6
