Commit message: Whole-body URDFs: origin at the soles, so z = 0 is the ground
base_link's origin was 19.9 mm above the soles, so a URDF loaded with its
origin on the floor (Isaac Lab, ROS, PyBullet) had its feet through it.
Both URDFs (hands and grippers) now put base_link at the soles; base_link
and the joints on it move up 19.9 mm, nothing else. The MuJoCo files are
rebuilt from them and are unchanged in effect: their soles were already
on the floor. No mesh changes.

Co-Authored-By: Wilson Cheng <150957380+wilsonchenghy@users.noreply.github.com>

File: assets/pioneer_whole_body_humanoid/pioneer_whole_body_humanoid.urdf (robot description, URDF)
Before this commit: robot pioneer_whole_body_humanoid, 70 links, 69 joints
Joints:
- joint Hip_F_L: origin xyz=0.084000 0.000000 0.828000 -> xyz=0.084000 0.000000 0.847917
- joint Hip_F_R: origin xyz=-0.084000 0.000000 0.828000 -> xyz=-0.084000 0.000000 0.847917
- joint waist_yaw: origin xyz=0.000000 0.000000 0.897000 -> xyz=0.000000 0.000000 0.916917

File: assets/pioneer_whole_body_humanoid/pioneer_whole_body_humanoid_gripper.urdf (robot description, URDF)
Before this commit: robot pioneer_whole_body_humanoid_gripper, 32 links, 31 joints
Joints:
- joint Hip_F_L: origin xyz=0.084000 0.000000 0.828000 -> xyz=0.084000 0.000000 0.847917
- joint Hip_F_R: origin xyz=-0.084000 0.000000 0.828000 -> xyz=-0.084000 0.000000 0.847917
- joint waist_yaw: origin xyz=0.000000 0.000000 0.897000 -> xyz=0.000000 0.000000 0.916917

Commit message: Whole-body models: real joint limits, estimated masses, motion checks
Every joint had a placeholder 10 Nm / 6 rad/s limit and the robot weighed
6.6 kg, so torque-driven motion in a simulator came out wrong. Each joint
now carries its motor's effort and velocity (legs and arms exact; waist,
neck and the hands' wrist / fingers estimates). Each link's mass, centre of
mass and inertia are summed from its CAD parts, motors at their datasheet
weights: 44.7 kg (hands), 42.2 kg (grippers), estimates. The ankle cross,
a near-massless placeholder between two 60 Nm motors, is a 0.1 kg block.

to_mjcf.py caps each actuator at its motor's effort. check_hold.py and
check_motion.py test that the motors hold the robot up and that every joint
moves cleanly; check_leg_directions.py tracks a toe point on the foot.

Co-Authored-By: Wilson Cheng <150957380+wilsonchenghy@users.noreply.github.com>

File: assets/pioneer_whole_body_humanoid/pioneer_whole_body_humanoid.urdf (robot description, URDF)
Before this commit: robot pioneer_whole_body_humanoid, 70 links, 69 joints
Links:
- link base_link: mass 0.2439 -> 4.6735
- link head: mass 0.2599 -> 0.5348
- link l_ankle_cross: mass 0.0100 -> 0.1000
- link l_arm_link1: mass 0.3313 -> 1.3298
- link l_arm_link2: mass 0.1719 -> 0.7890
- link l_arm_link3: mass 0.2121 -> 0.8487
- link l_arm_link4: mass 0.0788 -> 0.6014
- link l_foot: mass 0.1397 -> 1.0778
- link l_forearm: mass 0.0818 -> 1.4841
- link l_hand_D: mass 0.0100 -> 0.0060
- link l_hand_D_I: mass 0.0100 -> 0.0060
- link l_hand_D_L: mass 0.0100 -> 0.0060
- link l_hand_D_R: mass 0.0100 -> 0.0060
- link l_hand_H: mass 0.0454 -> 0.0880
- link l_hand_I: mass 0.0100 -> 0.0027
- link l_hand_I_I: mass 0.0100 -> 0.0027
- link l_hand_I_L: mass 0.0100 -> 0.0027
- link l_hand_I_R: mass 0.0100 -> 0.0027
- link l_hand_P: mass 0.0100 -> 0.0084
- link l_hand_P_I: mass 0.0100 -> 0.0084
- link l_hand_P_L: mass 0.0100 -> 0.0084
- link l_hand_P_R: mass 0.0100 -> 0.0084
- link l_hand_TC: mass 0.0100 -> 0.0066
- link l_hand_TD: mass 0.0100 -> 0.0032
- link l_hand_TF: mass 0.0100 -> 0.0036
- link l_hand_TP: mass 0.0100 -> 0.0055
- link l_hand_U: mass 0.0100 -> 0.0050
- link l_hand_U_I: mass 0.0100 -> 0.0050
- link l_hand_U_L: mass 0.0100 -> 0.0050
- link l_hand_U_R: mass 0.0100 -> 0.0050
- link l_hand_W: mass 0.0161 -> 0.0486
- link l_hip_pitch_link: mass 0.1980 -> 1.3125
- link l_hip_roll_link: mass 0.2332 -> 1.5837
- link l_shank_foot: mass 0.4993 -> 4.8588
- link l_thigh: mass 0.3566 -> 2.8299
- link neck_link: mass 0.1074 -> 0.1994
- link r_ankle_cross: mass 0.0100 -> 0.1000
- link r_arm_link1: mass 0.3313 -> 1.3298
- link r_arm_link2: mass 0.1798 -> 0.7890
- link r_arm_link3: mass 0.2121 -> 0.8487
- link r_arm_link4: mass 0.0788 -> 0.6014
- link r_foot: mass 0.1397 -> 1.0778
- link r_forearm: mass 0.0818 -> 1.4841
- link r_hand_D: mass 0.0100 -> 0.0060
- link r_hand_D_I: mass 0.0100 -> 0.0060
- link r_hand_D_L: mass 0.0100 -> 0.0060
- link r_hand_D_R: mass 0.0100 -> 0.0060
- link r_hand_H: mass 0.0454 -> 0.0880
- link r_hand_I: mass 0.0100 -> 0.0027
- link r_hand_I_I: mass 0.0100 -> 0.0027
- link r_hand_I_L: mass 0.0100 -> 0.0027
- link r_hand_I_R: mass 0.0100 -> 0.0027
- link r_hand_P: mass 0.0100 -> 0.0084
- link r_hand_P_I: mass 0.0100 -> 0.0084
- link r_hand_P_L: mass 0.0100 -> 0.0084
- link r_hand_P_R: mass 0.0100 -> 0.0084
- link r_hand_TC: mass 0.0100 -> 0.0066
- link r_hand_TD: mass 0.0100 -> 0.0032
- link r_hand_TF: mass 0.0100 -> 0.0036
- link r_hand_TP: mass 0.0100 -> 0.0055
- link r_hand_U: mass 0.0100 -> 0.0050
- link r_hand_U_I: mass 0.0100 -> 0.0050
- link r_hand_U_L: mass 0.0100 -> 0.0050
- link r_hand_U_R: mass 0.0100 -> 0.0050
- link r_hand_W: mass 0.0161 -> 0.0486
- link r_hip_pitch_link: mass 0.1980 -> 1.3125
- link r_hip_roll_link: mass 0.2332 -> 1.5837
- link r_shank_foot: mass 0.4993 -> 4.8588
- link r_thigh: mass 0.3566 -> 2.8299
- link torso: mass 1.2415 -> 5.1662
Joints:
- joint Ankle_P_L: limit lower=-0.5236 upper=0.8727 effort=10 velocity=6 -> lower=-0.5236 upper=0.8727 effort=60 velocity=20.42
- joint Ankle_P_R: limit lower=-0.5236 upper=0.8727 effort=10 velocity=6 -> lower=-0.5236 upper=0.8727 effort=60 velocity=20.42
- joint Ankle_R_L: limit lower=-0.2618 upper=0.2618 effort=10 velocity=6 -> lower=-0.2618 upper=0.2618 effort=60 velocity=20.42
- joint Ankle_R_R: limit lower=-0.2618 upper=0.2618 effort=10 velocity=6 -> lower=-0.2618 upper=0.2618 effort=60 velocity=20.42
- joint Hip_A_L: limit lower=-0.1745 upper=1.0472 effort=10 velocity=6 -> lower=-0.1745 upper=1.0472 effort=120 velocity=20.944
- joint Hip_A_R: limit lower=-0.1745 upper=1.0472 effort=10 velocity=6 -> lower=-0.1745 upper=1.0472 effort=120 velocity=20.944
- joint Hip_F_L: limit lower=-0.3491 upper=1.5708 effort=10 velocity=6 -> lower=-0.3491 upper=1.5708 effort=222 velocity=3.6652
- joint Hip_F_R: limit lower=-0.3491 upper=1.5708 effort=10 velocity=6 -> lower=-0.3491 upper=1.5708 effort=222 velocity=3.6652
- joint Hip_R_L: limit lower=-0.5236 upper=1.5708 effort=10 velocity=6 -> lower=-0.5236 upper=1.5708 effort=60 velocity=20.42
- joint Hip_R_R: limit lower=-0.5236 upper=1.5708 effort=10 velocity=6 -> lower=-0.5236 upper=1.5708 effort=60 velocity=20.42
- joint Knee_L: limit lower=-1.1345 upper=0.0000 effort=10 velocity=6 -> lower=-1.1345 upper=0.0000 effort=222 velocity=3.6652
- joint Knee_R: limit lower=-1.1345 upper=0.0000 effort=10 velocity=6 -> lower=-1.1345 upper=0.0000 effort=222 velocity=3.6652
- joint l_abd: limit lower=-0.2618 upper=0.2618 effort=10 velocity=6 -> lower=-0.2618 upper=0.2618 effort=0.5 velocity=6
- joint l_dip: limit lower=0.0000 upper=1.5708 effort=10 velocity=6 -> lower=0.0000 upper=1.5708 effort=0.5 velocity=6
- joint l_elbow: limit lower=-1.5708 upper=1.5708 effort=10 velocity=6 -> lower=-1.5708 upper=1.5708 effort=22 velocity=6
- joint l_forearm_roll: limit lower=-1.5708 upper=1.5708 effort=10 velocity=6 -> lower=-1.5708 upper=1.5708 effort=22 velocity=6
- joint l_i_abd: limit lower=-0.2618 upper=0.2618 effort=10 velocity=6 -> lower=-0.2618 upper=0.2618 effort=0.5 velocity=6
- joint l_i_dip: limit lower=0.0000 upper=1.5708 effort=10 velocity=6 -> lower=0.0000 upper=1.5708 effort=0.5 velocity=6
- joint l_i_mcp: limit lower=0.0000 upper=1.5708 effort=10 velocity=6 -> lower=0.0000 upper=1.5708 effort=0.5 velocity=6
- joint l_i_pip: limit lower=0.0000 upper=1.5708 effort=10 velocity=6 -> lower=0.0000 upper=1.5708 effort=0.5 velocity=6
- joint l_l_abd: limit lower=-0.2618 upper=0.2618 effort=10 velocity=6 -> lower=-0.2618 upper=0.2618 effort=0.5 velocity=6
- joint l_l_dip: limit lower=0.0000 upper=1.5708 effort=10 velocity=6 -> lower=0.0000 upper=1.5708 effort=0.5 velocity=6
- joint l_l_mcp: limit lower=0.0000 upper=1.5708 effort=10 velocity=6 -> lower=0.0000 upper=1.5708 effort=0.5 velocity=6
- joint l_l_pip: limit lower=0.0000 upper=1.5708 effort=10 velocity=6 -> lower=0.0000 upper=1.5708 effort=0.5 velocity=6
- joint l_mcp: limit lower=0.0000 upper=1.5708 effort=10 velocity=6 -> lower=0.0000 upper=1.5708 effort=0.5 velocity=6
- joint l_pip: limit lower=0.0000 upper=1.5708 effort=10 velocity=6 -> lower=0.0000 upper=1.5708 effort=0.5 velocity=6
- joint l_r_abd: limit lower=-0.2618 upper=0.2618 effort=10 velocity=6 -> lower=-0.2618 upper=0.2618 effort=0.5 velocity=6
- joint l_r_dip: limit lower=0.0000 upper=1.5708 effort=10 velocity=6 -> lower=0.0000 upper=1.5708 effort=0.5 velocity=6
- joint l_r_mcp: limit lower=0.0000 upper=1.5708 effort=10 velocity=6 -> lower=0.0000 upper=1.5708 effort=0.5 velocity=6
- joint l_r_pip: limit lower=0.0000 upper=1.5708 effort=10 velocity=6 -> lower=0.0000 upper=1.5708 effort=0.5 velocity=6
- joint l_shoulder_pitch: limit lower=-3.1416 upper=3.1416 effort=10 velocity=6 -> lower=-3.1416 upper=3.1416 effort=53 velocity=6
- joint l_shoulder_roll: limit lower=-1.5708 upper=1.5708 effort=10 velocity=6 -> lower=-1.5708 upper=1.5708 effort=53 velocity=6
- joint l_th_c: limit lower=0.0000 upper=0.8727 effort=10 velocity=6 -> lower=0.0000 upper=0.8727 effort=0.5 velocity=6
- joint l_th_f: limit lower=0.0000 upper=1.0472 effort=10 velocity=6 -> lower=0.0000 upper=1.0472 effort=0.5 velocity=6
- joint l_th_ip: limit lower=0.0000 upper=1.3963 effort=10 velocity=6 -> lower=0.0000 upper=1.3963 effort=0.5 velocity=6
- joint l_th_mcp: limit lower=0.0000 upper=1.3963 effort=10 velocity=6 -> lower=0.0000 upper=1.3963 effort=0.5 velocity=6
- joint l_upper_arm_yaw: limit lower=-1.5708 upper=1.5708 effort=10 velocity=6 -> lower=-1.5708 upper=1.5708 effort=22 velocity=6
- joint l_wrist_dev: limit lower=-0.3491 upper=0.5236 effort=10 velocity=6 -> lower=-0.3491 upper=0.5236 effort=2 velocity=6
- joint l_wrist_flex: limit lower=-1.0472 upper=1.0472 effort=10 velocity=6 -> lower=-1.0472 upper=1.0472 effort=2 velocity=6
- joint neck_pitch: limit lower=-0.3491 upper=0.5236 effort=10 velocity=6 -> lower=-0.3491 upper=0.5236 effort=5 velocity=6
- joint neck_yaw: limit lower=-1.2217 upper=1.2217 effort=10 velocity=6 -> lower=-1.2217 upper=1.2217 effort=5 velocity=6
- joint r_abd: limit lower=-0.2618 upper=0.2618 effort=10 velocity=6 -> lower=-0.2618 upper=0.2618 effort=0.5 velocity=6
- joint r_dip: limit lower=0.0000 upper=1.5708 effort=10 velocity=6 -> lower=0.0000 upper=1.5708 effort=0.5 velocity=6
- joint r_elbow: limit lower=-1.5708 upper=1.5708 effort=10 velocity=6 -> lower=-1.5708 upper=1.5708 effort=22 velocity=6
- joint r_forearm_roll: limit lower=-1.5708 upper=1.5708 effort=10 velocity=6 -> lower=-1.5708 upper=1.5708 effort=22 velocity=6
- joint r_i_abd: limit lower=-0.2618 upper=0.2618 effort=10 velocity=6 -> lower=-0.2618 upper=0.2618 effort=0.5 velocity=6
- joint r_i_dip: limit lower=0.0000 upper=1.5708 effort=10 velocity=6 -> lower=0.0000 upper=1.5708 effort=0.5 velocity=6
- joint r_i_mcp: limit lower=0.0000 upper=1.5708 effort=10 velocity=6 -> lower=0.0000 upper=1.5708 effort=0.5 velocity=6
- joint r_i_pip: limit lower=0.0000 upper=1.5708 effort=10 velocity=6 -> lower=0.0000 upper=1.5708 effort=0.5 velocity=6
- joint r_l_abd: limit lower=-0.2618 upper=0.2618 effort=10 velocity=6 -> lower=-0.2618 upper=0.2618 effort=0.5 velocity=6
- joint r_l_dip: limit lower=0.0000 upper=1.5708 effort=10 velocity=6 -> lower=0.0000 upper=1.5708 effort=0.5 velocity=6
- joint r_l_mcp: limit lower=0.0000 upper=1.5708 effort=10 velocity=6 -> lower=0.0000 upper=1.5708 effort=0.5 velocity=6
- joint r_l_pip: limit lower=0.0000 upper=1.5708 effort=10 velocity=6 -> lower=0.0000 upper=1.5708 effort=0.5 velocity=6
- joint r_mcp: limit lower=0.0000 upper=1.5708 effort=10 velocity=6 -> lower=0.0000 upper=1.5708 effort=0.5 velocity=6
- joint r_pip: limit lower=0.0000 upper=1.5708 effort=10 velocity=6 -> lower=0.0000 upper=1.5708 effort=0.5 velocity=6
- joint r_r_abd: limit lower=-0.2618 upper=0.2618 effort=10 velocity=6 -> lower=-0.2618 upper=0.2618 effort=0.5 velocity=6
- joint r_r_dip: limit lower=0.0000 upper=1.5708 effort=10 velocity=6 -> lower=0.0000 upper=1.5708 effort=0.5 velocity=6
- joint r_r_mcp: limit lower=0.0000 upper=1.5708 effort=10 velocity=6 -> lower=0.0000 upper=1.5708 effort=0.5 velocity=6
- joint r_r_pip: limit lower=0.0000 upper=1.5708 effort=10 velocity=6 -> lower=0.0000 upper=1.5708 effort=0.5 velocity=6
- joint r_shoulder_pitch: limit lower=-3.1416 upper=3.1416 effort=10 velocity=6 -> lower=-3.1416 upper=3.1416 effort=53 velocity=6
- joint r_shoulder_roll: limit lower=-1.5708 upper=1.5708 effort=10 velocity=6 -> lower=-1.5708 upper=1.5708 effort=53 velocity=6
- joint r_th_c: limit lower=0.0000 upper=0.8727 effort=10 velocity=6 -> lower=0.0000 upper=0.8727 effort=0.5 velocity=6
- joint r_th_f: limit lower=0.0000 upper=1.0472 effort=10 velocity=6 -> lower=0.0000 upper=1.0472 effort=0.5 velocity=6
- joint r_th_ip: limit lower=0.0000 upper=1.3963 effort=10 velocity=6 -> lower=0.0000 upper=1.3963 effort=0.5 velocity=6
- joint r_th_mcp: limit lower=0.0000 upper=1.3963 effort=10 velocity=6 -> lower=0.0000 upper=1.3963 effort=0.5 velocity=6
- joint r_upper_arm_yaw: limit lower=-1.5708 upper=1.5708 effort=10 velocity=6 -> lower=-1.5708 upper=1.5708 effort=22 velocity=6
- joint r_wrist_dev: limit lower=-0.3491 upper=0.5236 effort=10 velocity=6 -> lower=-0.3491 upper=0.5236 effort=2 velocity=6
- joint r_wrist_flex: limit lower=-1.0472 upper=1.0472 effort=10 velocity=6 -> lower=-1.0472 upper=1.0472 effort=2 velocity=6
- joint waist_yaw: limit lower=-1.5708 upper=1.5708 effort=10 velocity=6 -> lower=-1.5708 upper=1.5708 effort=60 velocity=6

File: assets/pioneer_whole_body_humanoid/pioneer_whole_body_humanoid_gripper.urdf (robot description, URDF)
Before this commit: robot pioneer_whole_body_humanoid_gripper, 32 links, 31 joints
Links:
- link base_link: mass 0.2439 -> 4.6735
- link head: mass 0.2599 -> 0.5348
- link l_ankle_cross: mass 0.0100 -> 0.1000
- link l_arm_link1: mass 0.3313 -> 1.3298
- link l_arm_link2: mass 0.1719 -> 0.7890
- link l_arm_link3: mass 0.2121 -> 0.8487
- link l_arm_link4: mass 0.0788 -> 0.6014
- link l_arm_link5: mass 0.0911 -> 0.2649
- link l_arm_link6: mass 0.0422 -> 0.1619
- link l_arm_link7: mass 0.0131 -> 0.0243
- link l_arm_link8: mass 0.0131 -> 0.0243
- link l_foot: mass 0.1397 -> 1.0778
- link l_hip_pitch_link: mass 0.1980 -> 1.3125
- link l_hip_roll_link: mass 0.2332 -> 1.5837
- link l_shank_foot: mass 0.4993 -> 4.8588
- link l_thigh: mass 0.3566 -> 2.8299
- link neck_link: mass 0.1074 -> 0.1994
- link r_ankle_cross: mass 0.0100 -> 0.1000
- link r_arm_link1: mass 0.3313 -> 1.3298
- link r_arm_link2: mass 0.1798 -> 0.7890
- link r_arm_link3: mass 0.2121 -> 0.8487
- link r_arm_link4: mass 0.0788 -> 0.6014
- link r_arm_link5: mass 0.0911 -> 0.2649
- link r_arm_link6: mass 0.0422 -> 0.1619
- link r_arm_link7: mass 0.0131 -> 0.0243
- link r_arm_link8: mass 0.0131 -> 0.0243
- link r_foot: mass 0.1397 -> 1.0778
- link r_hip_pitch_link: mass 0.1980 -> 1.3125
- link r_hip_roll_link: mass 0.2332 -> 1.5837
- link r_shank_foot: mass 0.4993 -> 4.8588
- link r_thigh: mass 0.3566 -> 2.8299
- link torso: mass 1.2415 -> 5.1662
Joints:
- joint Ankle_P_L: limit lower=-0.5236 upper=0.8727 effort=10 velocity=6 -> lower=-0.5236 upper=0.8727 effort=60 velocity=20.42
- joint Ankle_P_R: limit lower=-0.5236 upper=0.8727 effort=10 velocity=6 -> lower=-0.5236 upper=0.8727 effort=60 velocity=20.42
- joint Ankle_R_L: limit lower=-0.2618 upper=0.2618 effort=10 velocity=6 -> lower=-0.2618 upper=0.2618 effort=60 velocity=20.42
- joint Ankle_R_R: limit lower=-0.2618 upper=0.2618 effort=10 velocity=6 -> lower=-0.2618 upper=0.2618 effort=60 velocity=20.42
- joint Hip_A_L: limit lower=-0.1745 upper=1.0472 effort=10 velocity=6 -> lower=-0.1745 upper=1.0472 effort=120 velocity=20.944
- joint Hip_A_R: limit lower=-0.1745 upper=1.0472 effort=10 velocity=6 -> lower=-0.1745 upper=1.0472 effort=120 velocity=20.944
- joint Hip_F_L: limit lower=-0.3491 upper=1.5708 effort=10 velocity=6 -> lower=-0.3491 upper=1.5708 effort=222 velocity=3.6652
- joint Hip_F_R: limit lower=-0.3491 upper=1.5708 effort=10 velocity=6 -> lower=-0.3491 upper=1.5708 effort=222 velocity=3.6652
- joint Hip_R_L: limit lower=-0.5236 upper=1.5708 effort=10 velocity=6 -> lower=-0.5236 upper=1.5708 effort=60 velocity=20.42
- joint Hip_R_R: limit lower=-0.5236 upper=1.5708 effort=10 velocity=6 -> lower=-0.5236 upper=1.5708 effort=60 velocity=20.42
- joint Knee_L: limit lower=-1.1345 upper=0.0000 effort=10 velocity=6 -> lower=-1.1345 upper=0.0000 effort=222 velocity=3.6652
- joint Knee_R: limit lower=-1.1345 upper=0.0000 effort=10 velocity=6 -> lower=-1.1345 upper=0.0000 effort=222 velocity=3.6652
- joint joint1: limit lower=-2.3038 upper=1.7802 effort=10 velocity=6 -> lower=-2.3038 upper=1.7802 effort=53 velocity=6
- joint joint1L: limit lower=-2.3038 upper=1.7802 effort=10 velocity=6 -> lower=-2.3038 upper=1.7802 effort=53 velocity=6
- joint joint2: limit lower=-1.5708 upper=0.3491 effort=10 velocity=6 -> lower=-1.5708 upper=0.3491 effort=53 velocity=6
- joint joint2l: limit lower=-0.3491 upper=1.5708 effort=10 velocity=6 -> lower=-0.3491 upper=1.5708 effort=53 velocity=6
- joint joint3: limit lower=-1.3963 upper=3.7263 effort=10 velocity=6 -> lower=-1.3963 upper=3.7263 effort=22 velocity=6
- joint joint3l: limit lower=-3.7263 upper=1.3963 effort=10 velocity=6 -> lower=-3.7263 upper=1.3963 effort=22 velocity=6
- joint joint4: limit lower=-1.7453 upper=2.3126 effort=10 velocity=6 -> lower=-1.7453 upper=2.3126 effort=22 velocity=6
- joint joint4l: limit lower=-2.3126 upper=1.7453 effort=10 velocity=6 -> lower=-2.3126 upper=1.7453 effort=22 velocity=6
- joint joint5: limit lower=-4.3284 upper=1.3160 effort=10 velocity=6 -> lower=-4.3284 upper=1.3160 effort=22 velocity=6
- joint joint5l: limit lower=-1.3160 upper=4.3284 effort=10 velocity=6 -> lower=-1.3160 upper=4.3284 effort=22 velocity=6
- joint joint6: limit lower=-6.2832 upper=6.2832 effort=10 velocity=6 -> lower=-6.2832 upper=6.2832 effort=0.73 velocity=6
- joint joint6l: limit lower=-6.2832 upper=6.2832 effort=10 velocity=6 -> lower=-6.2832 upper=6.2832 effort=0.73 velocity=6
- joint joint7: limit lower=-0.0532 upper=0.0168 effort=10 velocity=6 -> lower=-0.0532 upper=0.0168 effort=30 velocity=0.2
- joint joint7l: limit lower=-0.0532 upper=0.0168 effort=10 velocity=6 -> lower=-0.0532 upper=0.0168 effort=30 velocity=0.2
- joint joint8: limit lower=-0.0132 upper=0.0468 effort=10 velocity=6 -> lower=-0.0132 upper=0.0468 effort=30 velocity=0.2
- joint joint8l: limit lower=-0.0132 upper=0.0468 effort=10 velocity=6 -> lower=-0.0132 upper=0.0468 effort=30 velocity=0.2
- joint neck_pitch: limit lower=-0.3491 upper=0.5236 effort=10 velocity=6 -> lower=-0.3491 upper=0.5236 effort=5 velocity=6
- joint neck_yaw: limit lower=-1.2217 upper=1.2217 effort=10 velocity=6 -> lower=-1.2217 upper=1.2217 effort=5 velocity=6
- joint waist_yaw: limit lower=-1.5708 upper=1.5708 effort=10 velocity=6 -> lower=-1.5708 upper=1.5708 effort=60 velocity=6

Commit message: Pioneer whole-body model: the elbow bends 125 deg
The elbow's lower (bend) limit goes from -90 to -125 deg in the URDF and MJCF. The real
elbow is said to reach 145 deg, but in the CAD model the forearm hits the upper-arm
housing from 129 deg (32 mm into it at 145), so 125 stays clear of that.

File: assets/pioneer_whole_body_humanoid/pioneer_whole_body_humanoid.urdf (robot description, URDF)
Before this commit: robot pioneer_whole_body_humanoid, 70 links, 69 joints
Joints:
- joint l_elbow: limit lower=-1.5708 upper=1.5708 effort=22 velocity=6 -> lower=-2.1817 upper=1.5708 effort=22 velocity=6
- joint r_elbow: limit lower=-1.5708 upper=1.5708 effort=22 velocity=6 -> lower=-2.1817 upper=1.5708 effort=22 velocity=6
