Commit message: Pioneer models: the knee bends 140 deg
The knee range was 65 deg (-1.1345 rad) in every Pioneer model; the real knee bends 140 deg (-2.4435 rad).
Updated in the leg-only and whole-body URDFs and their MJCFs (joint range and actuator ctrlrange).

File: assets/pioneer_leg_only_humanoid/pioneer_leg_only_humanoid.urdf (robot description, URDF)
Before this commit: robot pioneer_leg_only_humanoid, 16 links, 15 joints
Joints:
- joint Knee_L: limit lower=-1.1345 upper=0.0000 effort=222 velocity=3.6652 -> lower=-2.4435 upper=0.0000 effort=222 velocity=3.6652
- joint Knee_R: limit lower=-1.1345 upper=0.0000 effort=222 velocity=3.6652 -> lower=-2.4435 upper=0.0000 effort=222 velocity=3.6652

File: assets/pioneer_whole_body_humanoid/pioneer_whole_body_humanoid.urdf (robot description, URDF)
Before this commit: robot pioneer_whole_body_humanoid, 70 links, 69 joints
Joints:
- joint Knee_L: limit lower=-1.1345 upper=0.0000 effort=222 velocity=3.6652 -> lower=-2.4435 upper=0.0000 effort=222 velocity=3.6652
- joint Knee_R: limit lower=-1.1345 upper=0.0000 effort=222 velocity=3.6652 -> lower=-2.4435 upper=0.0000 effort=222 velocity=3.6652

File: assets/pioneer_whole_body_humanoid/pioneer_whole_body_humanoid_gripper.urdf (robot description, URDF)
Before this commit: robot pioneer_whole_body_humanoid_gripper, 32 links, 31 joints
Joints:
- joint Knee_L: limit lower=-1.1345 upper=0.0000 effort=222 velocity=3.6652 -> lower=-2.4435 upper=0.0000 effort=222 velocity=3.6652
- joint Knee_R: limit lower=-1.1345 upper=0.0000 effort=222 velocity=3.6652 -> lower=-2.4435 upper=0.0000 effort=222 velocity=3.6652
