Commit message: Replace Arm V2 forearms and grippers with articulated keyboard simulation

File: assets/pioneer_bimanual_arm/urdf/pioneer_bimanual_arm.urdf (robot description, URDF)
Before this commit: robot armv2URDF, 17 links, 16 joints
Links:
- added link left_bar0; visual mesh filename=package://armv2URDF/meshes/left_new_wrist_01_hum_arm_grippe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
- added link left_bar1; visual mesh filename=package://armv2URDF/meshes/left_new_wrist_02_hum_arm_grippe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
- added link left_crank; visual mesh filename=package://armv2URDF/meshes/left_new_wrist_03_grippermotorar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
- added link right_bar0; visual mesh filename=package://armv2URDF/meshes/right_new_wrist_01_hum_arm_gripp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
- added link right_bar1; visual mesh filename=package://armv2URDF/meshes/right_new_wrist_02_hum_arm_gripp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
- added link right_crank; visual mesh filename=package://armv2URDF/meshes/right_new_wrist_03_grippermotora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
- link base_link: mass 9.70005004618049 -> None; geometry visual mesh filename=package://armv2URDF/meshes/original_241_shoulderbearinghold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; visual mesh filename=package://armv2URDF/meshes/original_242_arm12bearing_csk_fo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
- link link1: mass 0.946680841893098 -> None; geometry visual mesh filename=package://armv2URDF/meshes/original_005_arm12rotor_fillet1.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; visual mesh filename=package://armv2URDF/meshes/original_006_arm12v2_boss_extrud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
- link link1L: mass 0.946692068071669 -> None; geometry visual mesh filename=package://armv2URDF/meshes/original_014_mirrorarm12v2_arm12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; visual mesh filename=package://armv2URDF/meshes/original_015_arm12spider_fillet5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
- link link2: mass 0.524797758723649 -> None; geometry visual mesh filename=package://armv2URDF/meshes/original_185_arm23v2bearingmount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; visual mesh filename=package://armv2URDF/meshes/original_186_arm23v2_cut_extrude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
- link link2l: mass 0.524798985890022 -> None; geometry visual mesh filename=package://armv2URDF/meshes/original_074_mirrorarm23v2bearin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; visual mesh filename=package://armv2URDF/meshes/original_075_mirrorarm23v2_arm23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
- link link3: mass 0.617876375655755 -> None; geometry visual mesh filename=package://armv2URDF/meshes/original_380_arm34v2base_none.stl; visual mesh filename=package://armv2URDF/meshes/original_381_arm34v2base_none.stl
- link link3l: mass 0.61786854410098 -> None; geometry visual mesh filename=package://armv2URDF/meshes/original_324_mirrorarm34v2cover_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; visual mesh filename=package://armv2URDF/meshes/original_325_mirrorarm34v2base_a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
- link link4: mass 0.236099727990138 -> None; geometry visual mesh filename=package://armv2URDF/meshes/original_130_arm45v2_cut_extrude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; visual mesh filename=package://armv2URDF/meshes/original_131_ak80_motor_none.stl
- link link4l: mass 0.23609959618399 -> None; geometry visual mesh filename=package://armv2URDF/meshes/original_019_mirrorarm45v2_arm45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; visual mesh filename=package://armv2URDF/meshes/original_020_mirrorak80_motor_no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
- link link5: mass 0.260193841211252 -> None; geometry visual mesh filename=package://armv2URDF/meshes/original_003_gl40iistat_none.stl; visual mesh filename=package://armv2URDF/meshes/original_004_gl40iistat_none.stl
- link link5l: mass 0.260192598192353 -> None; geometry visual mesh filename=package://armv2URDF/meshes/left_new_cover_1.stl; visual mesh filename=package://armv2URDF/meshes/left_new_forearm_1.stl
- link link6: mass 0.120420205315175 -> None; geometry visual mesh filename=package://armv2URDF/meshes/original_012_gl40iirot_none.stl; visual mesh filename=package://armv2URDF/meshes/original_013_gl40iirot_none.stl
- link link6l: mass 0.120420993331066 -> None; geometry visual mesh filename=package://armv2URDF/meshes/left_new_wrist_07_0710_wrist_dua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; visual mesh filename=package://armv2URDF/meshes/left_new_wrist_08_hum_arm_grippe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
- link link7: mass 0.0372930675250569 -> None; geometry visual mesh filename=package://armv2URDF/meshes/right_new_wrist_04_left_finger_1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; visual mesh filename=package://armv2URDF/meshes/right_new_wrist_05_left_finger_1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
- link link7l: mass 0.0372932549660758 -> None; geometry visual mesh filename=package://armv2URDF/meshes/left_new_wrist_04_left_finger_1_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; visual mesh filename=package://armv2URDF/meshes/left_new_wrist_05_left_finger_1_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
- link link8: mass 0.0372930675242417 -> None; geometry visual mesh filename=package://armv2URDF/meshes/right_new_wrist_15_hum_arm_gripp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; visual mesh filename=package://armv2URDF/meshes/right_new_wrist_16_right_finger_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
- link link8l: mass 0.0372932549731019 -> None; geometry visual mesh filename=package://armv2URDF/meshes/left_new_wrist_15_hum_arm_grippe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; visual mesh filename=package://armv2URDF/meshes/left_new_wrist_16_right_finger_1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
Joints:
- added joint left_gripper: type revolute, parent link6l, child left_crank, origin xyz=1.60010893424e-14 1.39888101103e-14 -0.0953113883009 rpy=0 0 0, axis 0 0 1, limit lower=-0.17453292519943295 upper=1.5707963267948966 effort=100 velocity=1
- added joint left_linkage_pin0: type revolute, parent left_crank, child left_bar0, origin xyz=-0.0259779008051 -0.0150049548403 -0.0125 rpy=0 0 0, axis 0 0 1, limit lower=-6.283185307179586 upper=6.283185307179586 effort=100 velocity=1
- added joint left_linkage_pin1: type revolute, parent left_crank, child left_bar1, origin xyz=0.0259779008051 0.0150049548403 -0.0125 rpy=0 0 0, axis 0 0 1, limit lower=-6.283185307179586 upper=6.283185307179586 effort=100 velocity=1
- added joint right_gripper: type revolute, parent link6, child right_crank, origin xyz=1.60010893424e-14 -1.39888101103e-14 -0.0953113883009 rpy=0 0 0, axis 0 0 -1, limit lower=-0.17453292519943295 upper=1.5707963267948966 effort=100 velocity=1
- added joint right_linkage_pin0: type revolute, parent right_crank, child right_bar0, origin xyz=-0.0259779008051 0.0150049548403 -0.0125 rpy=0 0 0, axis 0 0 -1, limit lower=-6.283185307179586 upper=6.283185307179586 effort=100 velocity=1
- added joint right_linkage_pin1: type revolute, parent right_crank, child right_bar1, origin xyz=0.0259779008051 -0.0150049548403 -0.0125 rpy=0 0 0, axis 0 0 -1, limit lower=-6.283185307179586 upper=6.283185307179586 effort=100 velocity=1
- joint joint1: limit lower=-2.303835 upper=1.780236 effort=0 velocity=0 -> lower=-1.7453292519943295 upper=1.7453292519943295 effort=100 velocity=1; origin xyz=0.0215734774382594 -0.163325 0.060481929205022 rpy=0 0 0 -> xyz=0.0215734774383 -0.163325 0.060481929205 rpy=0 0 0
- joint joint1L: limit lower=-2.303835 upper=1.780236 effort=0 velocity=0 -> lower=-1.7453292519943295 upper=1.7453292519943295 effort=100 velocity=1; origin xyz=0.0215734774382595 0.163325 0.060481929205022 rpy=0 0 0 -> xyz=0.0215734774383 0.163325 0.060481929205 rpy=0 0 0
- joint joint2: limit lower=-1.570796 upper=0.349066 effort=0 velocity=0 -> lower=-1.3089969389957472 upper=1.3089969389957472 effort=100 velocity=1; origin xyz=-0.0428200564481259 -0.116 -0.000180788468191695 rpy=0 0 0 -> xyz=-0.00702084238344 -0.116 0 rpy=0 0 0
- joint joint2l: limit lower=-0.349066 upper=1.570796 effort=0 velocity=0 -> lower=-1.3089969389957472 upper=1.3089969389957472 effort=100 velocity=1; origin xyz=-0.00882005644812602 0.116 -0.000180788468191695 rpy=0 0 0 -> xyz=-0.00702084238344 0.116 0 rpy=0 0 0
- joint joint3: limit lower=-1.396263 upper=3.726278 effort=0 velocity=0 -> lower=-2.0943951023931953 upper=2.0943951023931953 effort=100 velocity=1; origin xyz=0.0359999999999998 0 -0.1162999991972 rpy=0 0 0 -> xyz=0 0 -0.116299999197 rpy=0 0 0
- joint joint3l: limit lower=-3.726278 upper=1.396263 effort=0 velocity=0 -> lower=-2.0943951023931953 upper=2.0943951023931953 effort=100 velocity=1; origin xyz=0.00200000000000037 0 -0.117299999197201 rpy=0 0 0 -> xyz=0 0 -0.116299999197 rpy=0 0 0
- joint joint4: limit lower=-1.745329 upper=2.312561 effort=0 velocity=0 -> lower=-1.9198621771937625 upper=1.9198621771937625 effort=100 velocity=1; origin xyz=0 -0.0252499991972028 -0.1846 rpy=0 0 0 -> xyz=0 -0.0022500008028 -0.1846 rpy=0 0 0
- joint joint4l: limit lower=-2.312561 upper=1.745329 effort=0 velocity=0 -> lower=-1.9198621771937625 upper=1.9198621771937625 effort=100 velocity=1; origin xyz=0 0.025249999197197 -0.183599999999999 rpy=0 0 0 -> xyz=0 0.0022500008028 -0.1846 rpy=0 0 0
- joint joint5: limit lower=-4.328417 upper=1.315978 effort=0 velocity=0 -> lower=-3.141592653589793 upper=3.141592653589793 effort=100 velocity=1; origin xyz=0 0.0229999999999994 -0.1074999991972 rpy=0 0 0 -> xyz=0 0 -0.107499999197 rpy=0 0 0
- joint joint5l: limit lower=-1.315978 upper=4.328417 effort=0 velocity=0 -> lower=-3.141592653589793 upper=3.141592653589793 effort=100 velocity=1; origin xyz=0 -0.0230249983943991 -0.169243101839289 rpy=0 0 0 -> xyz=0 0 -0.107499999197 rpy=0 0 0
- joint joint6: limit lower=-6.283185 upper=6.283185 effort=0 velocity=0 -> lower=-1.5707963267948966 upper=1.5707963267948966 effort=100 velocity=1; origin xyz=0 0.037 -0.128000000000001 rpy=0 0 0 -> xyz=0 -0.007 -0.128 rpy=0 0 0
- joint joint6l: limit lower=-6.283185 upper=6.283185 effort=0 velocity=0 -> lower=-1.5707963267948966 upper=1.5707963267948966 effort=100 velocity=1; origin xyz=-2.28300451460273e-14 -0.0459750016055988 -0.0662568973579128 rpy=0 0 0 -> xyz=0 0.007 -0.128 rpy=0 0 0
- joint joint7: axis 0 -1 0 -> -1 -0 -0; limit lower=-0.0532 upper=0.0168 effort=0 velocity=0 -> lower=-0.040517261618092236 upper=0.0007105513753589827 effort=100 velocity=1; origin xyz=0 0.0261579738681254 -0.11101425916694 rpy=0 0 0 -> xyz=-0.0552110970681 0.0217444085457 -0.107811388301 rpy=0 0 0
- joint joint7l: axis 0 1 0 -> -1 -0 -0; limit lower=-0.0532 upper=0.0168 effort=0 velocity=0 -> lower=-0.040517261618092236 upper=0.0007105513753589827 effort=100 velocity=1; origin xyz=0 -0.0171579738681266 -0.11101425916694 rpy=0 0 0 -> xyz=-0.0552110970681 -0.0217444085457 -0.107811388301 rpy=0 0 0
- joint joint8: axis 0 -1 0 -> -1 -0 -0; limit lower=-0.0132 upper=0.0468 effort=0 velocity=0 -> lower=-0.0007098349346630607 upper=0.04051562268663317 effort=100 velocity=1; origin xyz=0 -0.0771579775183292 -0.116558517434743 rpy=0 0 0 -> xyz=0.0552100839797 -0.0217488014319 -0.107811388301 rpy=0 0 0
- joint joint8l: axis 0 1 0 -> -1 -0 -0; limit lower=-0.0132 upper=0.0468 effort=0 velocity=0 -> lower=-0.0007098349346630607 upper=0.04051562268663317 effort=100 velocity=1; origin xyz=0 0.0861579775183273 -0.116558517434743 rpy=0 0 0 -> xyz=0.0552100839797 0.0217488014319 -0.107811388301 rpy=0 0 0
